File: Hardware/CAD/XMICRO-SERIAL V1.0.brd (EAGLE design)
At the start: 203.2 x 101.6 mm, 95 parts, among them J1 D9-MPH, J2 D9-MPH, J3 MINI-DIN6, J4 PINHD1X3, J5 PINHD1X3, Q1 2N5088, Q2 2N5088, Q3 2N5088, U1 555, U10 74280, U11 74273, U12 74164, U13 74164, U14 7474, U15 74244, U16 74244, U17 74240, U18 74280, U19 74165, U2 7486, U20 74165, U21 74244, U22 7404, U23 74245, U24 16550, U25 16550, U26 75185, U27 75185, U28 7414, U29 TC962, U3 7410, U4 7404, U5 7474, U6 7474, U7 7408, U8 74138, U9 74138, Y1 1.8432MHz

Commit message: Initial commit for finalized V1.0
Parts:
- removed C39: 10uF, rcl:E2,5-5
- removed C40: 0.1uF, Custom:C100
- removed CE0: XMICRO-BUS-EDGE62M, Custom:EDGE62M
- removed J5: PINHD1X3, Custom:1X03
- removed JP5, JP6, JP7: PINHD-1X2THRU, Custom:1X02
- added C36, C37: 0.1uF, rcl:C025-024X044
- added P1: XMICRO-BUS-EDGE, XMICRO:EDGE62M
- added Q4: VN2106, transistor-misc:TO92
- added R10: 0, resistor:0207/10
- added RN2: 10, resistor-sil:SIL8
- added RN3: 10k, resistor-sil:SIL9
- C1, C10, C11, C12, C13, C14, C15, C16, C17, C18, C19, C2, C20, C21, C22, C23, C24, C25, C26, C27, C28, C3, C4, C5, C6, C7, C8, C9: device Custom:C100 -> rcl:C025-024X044
- C29: value 10nF -> 0.1uF; device Custom:C100 -> rcl:C025-024X044
- C30: value 0.1uF -> 10nF; device rcl:E2,5-6 -> rcl:C025-024X044
- C31: value 220uF -> 0.1uF; device Custom:C-10-5 -> rcl:C025-024X044
- C32: value 0.1uF -> 33uF; device Custom:C100 -> rcl:E2,5-6
- C33: value 0.1uF -> 10uF; device Custom:C100 -> rcl:E2,5-5
- J1, J2: value D9-MPH -> DSUB-9M-PH; device Custom:D9-H -> connector-misc:DSUB-9M-H
- J3: device Custom:MINI-DIN6 -> connector-misc:MINI-DIN6
- J4: value PINHD1X3 -> 1X3; device Custom:1X03 -> header:1X3
- JP1, JP2, JP3, JP4: value PINHD-1X2THRU -> 1X2-THRU; device Custom:1X02 -> header:1X2
- Q1, Q2, Q3: device Custom:TO92 -> transistor-misc:TO92
- R1, R2, R3, R8, R9: device resistor:0207/10 -> rcl:0207/10
- R4: value 10k -> 100k; device resistor:0207/10 -> rcl:0207/10
- R5: value 100k -> 10k; device resistor:0207/10 -> rcl:0207/10
- R6: value 10k -> 1.2k; device resistor:0207/10 -> rcl:0207/10
- R7: value 1.2k -> 10k; device resistor:0207/10 -> rcl:0207/10
- RN1: value 10k -> 10; device Custom:SIL9 -> resistor-sil:SIL8
- TP1, TP2: value PINHD-1X1 -> TP-040; device Custom:1X01 -> header:TP-040
- U10: value 74280 -> 74HCT280N
- U11: value 74273 -> 74HCT273N
- U12, U13: value 74164 -> 74HCT164N
- U14, U5, U6: value 7474 -> 74HCT74N
- U15: value 74244 -> 74HCT14N; device 74xx-us:DIL20 -> 74xx-us:DIL14
- U16: value 74244 -> 74HCT244N
- U17: value 74240 -> 74HCT244N
- U18: value 74280 -> 74HCT240N; device 74xx-us:DIL14 -> 74xx-us:DIL20
- U19: value 74165 -> 74HCT280N; device 74xx-us:DIL16 -> 74xx-us:DIL14
- U2: value 7486 -> 74HCT86N
- U20: value 74165 -> 74HCT165N
- U21: value 74244 -> 74HCT165N; device 74xx-us:DIL20 -> 74xx-us:DIL16
- U22: value 7404 -> 74ABT244N; device 74xx-eu:DIL14 -> 74xx-us:DIL20
- U23: value 74245 -> 74HCT04N; device 74xx-us:DIL20 -> 74xx-us:DIL14
- U24: value 16550 -> TC962; device Custom:S44 -> ic-misc:DIL8
- U25: value 16550 -> 74ABT245N; device Custom:S44 -> 74xx-us:DIL20
- U26, U27: value 75185 -> 16C550; device Custom:DIL20 -> ic-misc:S44
- U28: value 7414 -> 75185N; device 74xx-us:DIL14 -> ic-misc:DIL20
- U29: value TC962 -> 75185N; device Custom:DIL8 -> ic-misc:DIL20
- U3: value 7410 -> 74HCT10N
- U4: value 7404 -> 74HCT04N
- U7: value 7408 -> 74HCT08N
- U8, U9: value 74138 -> 74F138N; device 74xx-eu:DIL16 -> 74xx-us:DIL16
- Y1: device Custom:DIL08S -> crystal-misc:DIL08S
- moved C29 161.7 mm to (181.6, 60.6)
- moved C31 120.9 mm to (21.0, 83.8), turned to 0 degrees
- moved C28 94.6 mm to (181.6, 27.9), turned to 0 degrees
- moved U21 90.3 mm to (107.3, 94.0)
- moved C21 89.4 mm to (94.6, 94.0)
- moved U28 88.7 mm to (181.6, 43.2), turned to 90 degrees
- moved C32 83.5 mm to (118.1, 10.2)
- moved C25 75.3 mm to (157.0, 12.1), turned to 270 degrees
- moved C33 74.1 mm to (125.4, 49.5)
- moved RN1 68.8 mm to (171.4, 3.81)
- moved U25 62.3 mm to (171.4, 12.1)
- moved U29 51.7 mm to (181.6, 75.9), turned to 90 degrees
- moved U23 48.6 mm to (130.8, 36.8), turned to 270 degrees
- moved C23 45.8 mm to (130.8, 48.3), turned to 180 degrees
- moved JP3 42.1 mm to (42.5, 90.2), turned to 0 degrees
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- renumbered C38 to C35
Connections:
- removed net !INT_KB: JP3.1, U14.8
- removed net !IRQX: CE0.52, U22.12
- removed net GND: C1.P$2, C10.P$2, C11.P$2, C12.P$2, C13.P$2, C14.P$2, C15.P$2, C16.P$2, C17.P$2, C18.P$2, C19.P$2, C2.P$2, C20.P$2, C21.P$2, C22.P$2, C23.P$2, C24.P$2, C25.P$2, C26.P$2, C27.P$2, C28.P$2, C29.P$2, C3.P$2, C30.-, C31.-, C32.P$2, C33.P$2, C34.-, C39.+, C4.P$2, C40.P$2, C5.P$2, C6.P$2, C7.P$2, C8.P$2, C9.P$2, CE0.3, CE0.4, CE0.62, J1.P$5, J2.P$5, J3.3, J4.3, J5.3, JP4.1, JP5.1, JP6.1, JP7.1, Q1.1, Q2.1, Q3.1, R8.1, R9.1, U1.1, U10.1, U10.7, U11.10, U12.7, U13.7, U14.7, U15.10, U16.10, U16.17, U16.2, U16.4, U17.10, U18.7, U18.8, U19.5, U19.6, U19.8, U2.7, U20.8, U21.1, U21.10, U21.19, U22.7, U23.10, U24.21, U24.22, U24.25, U24.28, U25.21, U25.22, U25.25, U25.28, U26.11, U27.11, U28.7, U29.3, U3.7, U4.7, U5.7, U6.7, U7.7, U8.8, U9.8, Y1.4
- removed net ID0: U15.2
- removed net ID1: U15.17
- removed net ID2: U15.4
- removed net ID3: U15.15
- removed net ID4: U15.6
- removed net ID5: U15.13
- removed net ID6: U15.8
- removed net ID7: U15.11
- removed net N$112: U22.2, U24.14
- removed net N$122: J5.1, U25.38
- removed net N$123: J5.2, U25.35
- removed net N$125: J4.1, U24.38
- removed net N$136: J4.2, U24.35
- removed net SHIELD: J1.S1, J1.S2, J2.S1, J2.S2, J3.G$1, J3.G$2, J3.G$3, JP4.2, JP5.2, JP6.2, JP7.2
- removed net VCC: C1.P$1, C10.P$1, C11.P$1, C12.P$1, C13.P$1, C14.P$1, C15.P$1, C16.P$1, C17.P$1, C18.P$1, C19.P$1, C2.P$1, C20.P$1, C21.P$1, C22.P$1, C23.P$1, C24.P$1, C25.P$1, C26.P$1, C27.P$1, C28.P$1, C3.P$1, C31.+, C32.P$1, C33.P$1, C4.P$1, C5.P$1, C6.P$1, C7.P$1, C8.P$1, C9.P$1, CE0.5, CE0.6, J3.4, R1.2, R4.2, R6.2, R7.1, RN1.1, U1.4, U1.8, U10.14, U11.20, U12.14, U13.14, U14.10, U14.12, U14.14, U14.2, U14.4, U15.20, U16.20, U17.20, U18.14, U19.16, U2.10, U2.12, U2.13, U2.14, U2.4, U2.5, U2.9, U20.10, U20.11, U20.12, U20.13, U20.14, U20.16, U20.3, U21.20, U22.14, U22.5, U23.20, U24.44, U25.44, U26.20, U27.20, U28.14, U28.3, U3.14, U4.1, U4.14, U5.14, U5.2, U5.4, U6.10, U6.12, U6.14, U6.4, U7.12, U7.13, U7.14, U8.16, U9.16, Y1.1, Y1.8
- new net !BIRQX: P1.52, Q4.3
- new net !KB_INT_ENABLE: U23.13, U26.38
- new net +5V: C1.1, C10.1, C11.1, C12.1, C13.1, C14.1, C15.1, C16.1, C17.1, C18.1, C19.1, C2.1, C20.1, C21.1, C22.1, C23.1, C25.1, C26.1, C27.1, C28.1, C29.1, C3.1, C32.+, C36.1, C37.1, C4.1, C5.1, C6.1, C7.1, C8.1, C9.1, J3.4, P1.5, P1.6, R1.2, R5.2, R6.1, RN3.1, U1.4, U1.8, U10.14, U11.20, U12.14, U13.14, U14.10, U14.12, U14.14, U14.2, U14.4, U15.14, U15.3, U16.20, U16.4, U17.20, U18.20, U19.14, U2.10, U2.12, U2.13, U2.14, U2.4, U2.5, U2.9, U20.16, U21.10, U21.11, U21.12, U21.13, U21.14, U21.16, U21.3, U22.20, U23.14, U23.5, U25.20, U26.44, U27.44, U28.20, U29.20, U3.14, U4.14, U5.14, U5.2, U5.4, U6.10, U6.12, U6.14, U6.4, U7.14, U8.16, U9.16, Y1.1, Y1.8
- new net 0V: C1.2, C10.2, C11.2, C12.2, C13.2, C14.2, C15.2, C16.2, C17.2, C18.2, C19.2, C2.2, C20.2, C21.2, C22.2, C23.2, C24.2, C25.2, C26.2, C27.2, C28.2, C29.2, C3.2, C30.2, C31.2, C32.-, C33.-, C34.+, C36.2, C37.2, C4.2, C5.2, C6.2, C7.2, C8.2, C9.2, J1.5, J2.5, J3.3, J4.1, JP4.1, P1.21, P1.3, P1.4, P1.42, P1.62, Q1.1, Q2.1, Q3.1, Q4.1, R7.2, R8.1, R9.1, U1.1, U10.1, U10.7, U11.10, U12.7, U13.7, U14.7, U15.7, U16.10, U16.11, U16.13, U16.15, U16.17, U16.2, U16.6, U16.8, U17.10, U17.17, U17.2, U17.4, U18.10, U19.7, U19.8, U2.7, U20.5, U20.6, U20.8, U21.8, U22.1, U22.10, U22.19, U23.7, U24.3, U25.10, U26.21, U26.22, U26.25, U26.28, U27.21, U27.22, U27.25, U27.28, U28.11, U29.11, U3.7, U4.7, U5.7, U6.7, U7.7, U8.8, U9.8, Y1.4
- new net CGND: J1.S1, J1.S2, J2.S1, J2.S2, J3.G$1, J3.G$2, J3.G$3, JP4.2
- new net KB_DR: R3.1, U14.1, U14.9, U17.13, U7.12
- new net N$44: Q4.2, R10.2
- new net N$45: U3.13, U4.2
- new net N$46: U23.2, U26.14
- new net N$50: U23.12, U7.13
- new net N$51: J4.3, U27.38
- new net N$52: J4.2, U27.35
- new net N$53: RN2.2, U25.2
- new net N$54: RN2.4, U25.4
- new net N$55: RN2.6, U25.6
- new net N$56: RN2.8, U25.8
- new net N$57: P1.50, RN1.7
- new net N$58: P1.48, RN1.5
- new net N$59: P1.46, RN1.3
- new net N$68: P1.44, RN1.1
- net !BCSX: now also P1.9, U22.2; no longer CE0.9, U21.2
- net !BRD: now also P1.19, U22.4; no longer CE0.21, U21.4
- net !BRST: now also P1.10, U15.5; no longer CE0.14, U28.5
- net !BWR: now also P1.20, U22.17; no longer CE0.22, U21.17
- net !CSX: now also U22.18, U25.19, U26.16, U27.16; no longer U21.18, U23.19, U24.16, U25.16
- net !CS_IDR: now also U16.1, U16.19; no longer U15.1, U15.19
- net !CS_KBR: now also U18.1, U18.19; no longer U17.1, U17.19
- net !CS_KBW: now also U21.1; no longer U19.1
- net !CS_STR: now also U17.1, U17.19; no longer U16.1, U16.19
- net !KB_DATA: now also U15.12; no longer U28.12
- net !KB_WRCYCLE: now also U21.15; no longer U19.15
- net !RD: now also U22.16, U25.1, U26.24, U27.24; no longer U21.16, U23.1, U24.24, U25.24
- net !RST: now also U15.2; no longer U28.2
- net !WR: now also U22.3, U26.20, U27.20; no longer U21.3, U24.20, U25.20
- net +12V: now also C24.1, C33.+, P1.1, U24.8, U28.1, U29.1; no longer C34.+, C40.P$1, CE0.1, U26.1, U27.1, U29.8
- net -12V: now also C34.-, U24.5, U28.10, U29.10; no longer C39.-, U26.10, U27.10, U29.5
- net A0: now also U22.5, U26.31, U27.31; no longer U21.5, U24.31, U25.31
- net A1: now also U22.14, U26.30, U27.30; no longer U21.14, U24.30, U25.30
- net A2: now also U22.7, U26.29, U27.29; no longer U21.7, U24.29, U25.29
- net A3: now also U22.12, U23.1, U27.14; no longer U21.12, U22.1, U25.14
- net A4: now also U22.9, U23.3; no longer U21.9, U22.3
- net BA0: now also P1.22, U22.15; no longer CE0.23, U21.15
- net BA1: now also P1.23, U22.6; no longer CE0.24, U21.6
- net BA2: now also P1.24, U22.13; no longer CE0.25, U21.13
- net BA3: now also P1.25, U22.8; no longer CE0.26, U21.8
- net BA4: now also P1.26, U22.11; no longer CE0.27, U21.11
- net BUFF_KB_CLOCK: now also U15.8, U21.2; no longer U19.2, U28.8
- net D0: now also RN3.2, U18.18, U19.1, U20.4, U25.18, U26.2, U27.2; no longer RN1.2, U15.18, U18.1, U19.4, U23.18, U24.2, U25.2
- net D1: now also RN3.3, U18.3, U19.13, U20.3, U25.17, U26.3, U27.3; no longer RN1.3, U15.3, U18.13, U19.3, U23.17, U24.3, U25.3
- net D2: now also RN3.4, U18.16, U19.2, U20.14, U25.16, U26.4, U27.4; no longer RN1.4, U15.16, U18.2, U19.14, U23.16, U24.4, U25.4
- net D3: now also RN3.5, U18.5, U19.12, U20.13, U25.15, U26.5, U27.5; no longer RN1.5, U15.5, U18.12, U19.13, U23.15, U24.5, U25.5
- net D4: now also RN3.6, U18.14, U19.11, U20.12, U25.14, U26.6, U27.6; no longer RN1.6, U15.14, U18.11, U19.12, U23.14, U24.6, U25.6
- net D5: now also RN3.7, U18.7, U19.4, U20.11, U25.13, U26.7, U27.7; no longer RN1.7, U15.7, U18.4, U19.11, U23.13, U24.7, U25.7
- net D6: now also RN3.8, U18.12, U19.10, U21.6, U25.12, U26.8, U27.8; no longer RN1.8, U15.12, U18.10, U20.6, U23.12, U24.8, U25.8
- net D7: now also RN3.9, U19.9, U21.5, U25.11, U26.9, U27.9; no longer RN1.9, U15.9, U20.5, U23.11, U24.9, U25.9
- net INT_KB: now also JP3.1, U7.11; no longer R3.1, U14.1, U14.9, U16.13
- net INT_UART1: now also U17.11, U26.33; no longer U16.11, U24.33
- net INT_UART2: now also U17.8, U27.33; no longer U16.8, U25.33
- net KB_CLOCK: now also TP2.1, U15.11; no longer TP1.1, U28.11
- net KB_DATA: now also R5.1, TP1.1, U15.13; no longer R6.1, TP2.1, U28.13
- net KB_ERR: now also U17.6; no longer U16.6
- net KB_WRCYCLE: now also U17.15; no longer U16.15
- net N$1: now also J1.1, U28.2; no longer J1.P$1, U26.2
- net N$10: now also U26.43, U28.12; no longer U24.43, U26.12
- net N$103: now also R4.1; no longer R5.1
- net N$107: now also U23.10; no longer U22.10
- net N$11: now also U26.37, U28.13; no longer U24.37, U26.13
- net N$111: now also U20.10, U21.9; no longer U19.10, U20.9
- net N$114: now also U23.4, U26.15, U27.15; no longer U22.4, U24.15, U25.15
- net N$115: now also U23.9; no longer U22.9
- net N$116: now also U26.18, U27.18; no longer U24.18, U25.18
- net N$118: now also U23.11; no longer U22.11
- net N$12: now also U26.40, U28.14; no longer U24.40, U26.14
- net N$120: now also U19.5, U21.4; no longer U18.5, U20.4
- net N$124: now also R4.2; no longer R5.2
- net N$13: now also U26.13, U28.15; no longer U24.13, U26.15
- net N$133: now also C31.1, R6.2; no longer C30.+, R7.2
- net N$14: now also U26.36, U28.16; no longer U24.36, U26.16
- net N$140: now also C30.1; no longer C29.P$1
- net N$15: now also U26.11, U28.17; no longer U24.11, U26.17
- net N$16: now also U26.41, U28.18; no longer U24.41, U26.18
- net N$17: now also U26.42, U28.19; no longer U24.42, U26.19
- net N$18: now also U26.10, U26.17; no longer U24.10, U24.17
- net N$2: now also J1.2, U28.4; no longer J1.P$2, U26.4
- net N$21: now also R10.1; no longer U22.13
- net N$24: now also R7.1, U4.1; no longer R4.1, U3.13
- net N$25: now also U23.8; no longer U22.8
- net N$26: now also U15.10, U15.9; no longer U28.10, U28.9
- net N$27: now also U24.4; no longer U29.4
- net N$28: now also J2.2, U29.4; no longer J2.P$2, U27.4
- net N$29: now also J2.3, U29.6; no longer J2.P$3, U27.6
- net N$3: now also J1.3, U28.6; no longer J1.P$3, U26.6
- net N$30: now also J2.4, U29.8; no longer J2.P$4, U27.8
- net N$31: now also J2.6, U29.3; no longer J2.P$6, U27.3
- net N$32: now also J2.7, U29.5; no longer J2.P$7, U27.5
- net N$33: now also RN1.8, U25.9; no longer CE0.50, U23.9
- net N$34: now also P1.49, RN2.7; no longer CE0.49, U23.8
- net N$35: now also RN1.6, U25.7; no longer CE0.48, U23.7
- net N$36: now also P1.47, RN2.5; no longer CE0.47, U23.6
- net N$37: now also RN1.4, U25.5; no longer CE0.46, U23.5
- net N$38: now also P1.45, RN2.3; no longer CE0.45, U23.4
- net N$39: now also RN1.2, U25.3; no longer CE0.44, U23.3
- net N$4: now also J1.4, U28.8; no longer J1.P$4, U26.8
- net N$40: now also P1.43, RN2.1; no longer CE0.43, U23.2
- net N$41: now also J2.8, U29.7; no longer J2.P$8, U27.7
- net N$42: now also J2.9, U29.9; no longer J2.P$9, U27.9
- net N$43: now also U24.2; no longer U29.2
- net N$47: now also U27.43, U29.12; no longer U25.43, U27.12
- net N$48: now also U27.37, U29.13; no longer U25.37, U27.13
- net N$49: now also U27.40, U29.14; no longer U25.40, U27.14
- net N$5: now also J1.6, U28.3; no longer J1.P$6, U26.3
- net N$6: now also J1.7, U28.5; no longer J1.P$7, U26.5
- net N$60: now also U27.13, U29.15; no longer U25.13, U27.15
- net N$61: now also U27.36, U29.16; no longer U25.36, U27.16
- net N$62: now also U27.11, U29.17; no longer U25.11, U27.17
- net N$63: now also U27.41, U29.18; no longer U25.41, U27.18
- net N$64: now also U27.42, U29.19; no longer U25.42, U27.19
- net N$65: now also U27.10, U27.17; no longer U25.10, U25.17
- net N$7: now also J1.8, U28.7; no longer J1.P$8, U26.7
- net N$8: now also J1.9, U28.9; no longer J1.P$9, U26.9
- net N$86: now also U18.2; no longer U17.2
- net N$87: now also U20.9; no longer U19.9
- net N$9: now also J2.1, U29.2; no longer J2.P$1, U27.2
- net N$90: now also U18.17; no longer U17.17
- net N$91: now also U18.4; no longer U17.4
- net N$92: now also U18.15; no longer U17.15
- net N$94: now also U18.13; no longer U17.13
- net N$95: now also U18.8; no longer U17.8
- net N$96: now also U18.11; no longer U17.11
- net N$97: now also U18.6; no longer U17.6
- net N$99: now also U20.7; no longer U19.7
- net RST: now also U15.1, U15.6, U26.39, U27.39; no longer U24.39, U25.39, U28.1, U28.6
Routing:
- net VCC: track 1109.1 -> 0.00 mm, vias 24 -> 0
- net +5V: track 0.00 -> 1070.5 mm, vias 0 -> 21
- net KB_DR: track 0.00 -> 217.3 mm, vias 0 -> 5
- net INT_KB: track 188.6 -> 5.08 mm, vias 4 -> 0
- net N$50: track 0.00 -> 142.2 mm, vias 0 -> 2
- net !IRQX: track 90.9 -> 0.00 mm, vias 2 -> 0
- net GND: track 80.4 -> 0.00 mm, vias 62 -> 0
- net N$21: track 107.1 -> 179.1 mm, vias 1 -> 3
- net N$24: track 146.0 -> 79.1 mm, vias 1 -> 2
- net 0V: track 0.00 -> 43.5 mm, vias 0 -> 55
- net N$112: track 33.9 -> 0.00 mm, vias 1 -> 0
- net !KB_INT_ENABLE: track 0.00 -> 32.8 mm
- net N$46: track 0.00 -> 27.7 mm
- net N$52: track 0.00 -> 13.8 mm
- net N$123: track 13.8 -> 0.00 mm
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- added copper zone on layer 1, net 0V
- added copper zone on layer 16, net 0V
- added copper zone on layer 1, net CGND
- added copper zone on layer 16, net CGND
- added copper zone on layer 1, net LOGO-C
- added copper zone on layer 1, net LOGO-I
- added copper zone on layer 1, net LOGO-M
- added copper zone on layer 1, net LOGO-O
- added copper zone on layer 1, net LOGO-R
- added copper zone on layer 1, net LOGO-X
- removed copper zone on layer 1, net GND
- removed copper zone on layer 16, net GND
- removed copper zone on layer 1, net LOGO
- removed copper zone on layer 1, net S$1
- removed copper zone on layer 1, net SHIELD
- removed copper zone on layer 16, net SHIELD
Other:
- board text added: "CGND"
- board text added: "CHRIS WEIR ID $04"
- board text added: "PORT 1 INT"
- board text added: "PORT 2 INT"
- board text added: "V1.0 2410"
- board text removed: "0"
- board text removed: "1"
- board text removed: "2"
- board text removed: "3"
- board text removed: "4"
- board text removed: "5"
- board text removed: "6"
- board text removed: "7"
- board text removed: "CARD ID"
- board text removed: "CHRIS WEIR 2019"
- board text removed: "J1 INT"
- board text removed: "J2 INT"
- board text removed: "V1.1 1946"
